Commit message: Add GPS support and update EKF configurations for simulation

File: ora_description/description/dimensions.xacro (robot description, xacro)
@@ -35,4 +35,7 @@
   <xacro:property name="lidar_height" value="${71.7 * mm_to_m}"/>
   <xacro:property name="lidar_radius" value="${103.3 * mm_to_m / 2}"/>
+  <!-- GPS Dimensions -->
+  <xacro:property name="gps_height" value="${20 * mm_to_m}"/>
+  <xacro:property name="gps_radius" value="${50 * mm_to_m / 2}"/>
   <!-- Assorted Offset Values -->
   <xacro:property name="base_x_offset" value="${(back_caster_x_offset / 4)}"/>
@@ -40,3 +43,5 @@
   <xacro:property name="lidar_x_offset" value="${(base_length / 2) - (lidar_radius / 2) + (base_x_offset / 2)}"/>
   <xacro:property name="lidar_z_offset" value="${(base_height / 2) + (lidar_height / 2) + base_z_offset}"/>
+  <xacro:property name="gps_x_offset" value="${0}"/>
+  <xacro:property name="gps_z_offset" value="${(base_height / 2) + (gps_height / 2) + base_z_offset}"/>
 </robot>

File: ora_description/description/sensors.xacro (robot description, xacro)
@@ -65,4 +65,53 @@
     </sensor>
   </gazebo>
+  <!-- GPS -->
+  <link name="gps_link">
+    <inertial>
+      <origin xyz="0 0 0" rpy="0 0 0"/>
+      <mass value="0.125"/>
+      <inertia ixx="0.001" ixy="0" ixz="0" iyy="0.001" iyz="0" izz="0.001" />
+    </inertial>
+    <collision>
+      <origin xyz="0 0 0" rpy="0 0 0"/>
+      <geometry>
+        <cylinder radius="${gps_radius}" length="${gps_height}"/>
+      </geometry>
+    </collision>
+    <visual>
+      <origin xyz="0 0 0" rpy="0 0 0"/>
+      <geometry>
+        <cylinder radius="${gps_radius}" length="${gps_height}"/>
+      </geometry>
+    </visual>
+  </link>
+  <joint name="gps_joint" type="fixed">
+    <parent link="base_link"/>
+    <child link="gps_link"/>
+    <origin xyz="${gps_x_offset} 0 ${gps_z_offset}" rpy="0 0 0"/>
+  </joint>
+  <gazebo reference="gps_link">
+    <sensor name="navsat" type="navsat">
+      <always_on>true</always_on>
+      <update_rate>1</update_rate>
+      <topic>sim/gps/fix</topic>
+      <gz_frame_id>gps_link</gz_frame_id>
+      <navsat>
+        <position_sensing>
+          <horizontal>
+            <noise type="gaussian">
+              <mean>0.0</mean>
+              <stddev>0.0</stddev>
+            </noise>
+          </horizontal>
+          <vertical>
+            <noise type="gaussian">
+              <mean>0.0</mean>
+              <stddev>0.0</stddev>
+            </noise>
+          </vertical>
+        </position_sensing>
+      </navsat>
+    </sensor>
+  </gazebo>
   <!-- IMU -->
   <link name="imu_link">
